File: lemmy/lemmy.kicad_pcb (KiCad board)
At the start: 2 copper layers, 25 x 25 mm, 5 parts, among them J2 Conn_01x02

Commit message: traces
Parts:
- moved H1 101.1 mm to (85.2, 57.2)
- moved H3 101.1 mm to (85.3, 75.0)
- moved H4 101.1 mm to (67.6, 75.0)
- moved J2 101.1 mm to (85.7, 64.8)
- moved H2 101.1 mm to (67.6, 57.2)
Routing:
- net Net-(J1-Pin_2): track 0.00 -> 173.4 mm
- net Net-(J1-Pin_1): track 0.00 -> 137.6 mm
Other:
- board text removed: "PUSH BUTTON REV1.0"
- board text removed: "button space"

Commit message: redundancy
Routing:
- net Net-(J1-Pin_2): track 173.4 -> 185.9 mm
Changed lines of the file:
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@@
   (segment (start 68.638604 68.888604) (end 68.684188 68.888604) (width 0.5) (layer "F.Cu") (net 2))
   (segment (start 80.577208 69) (end 81.863604 67.713604) (width 0.5) (layer "F.Cu") (net 2))
-  (segment (start 67.35 62.45) (end 67.35 61.227208) (width 0.5) (layer "F.Cu") (net 2))
   (segment (start 69.83198 66.66802) (end 72.41802 66.66802) (width 0.5) (layer "F.Cu") (net 2))
   (segment (start 72.41802 66.66802) (end 72.95 67.2) (width 0.5) (layer "F.Cu") (net 2))
+  (segment (start 67.35 61.227208) (end 67.35 62.45) (width 0.5) (layer "F.Cu") (net 2))
   (segment (start 83.022792 74.4) (end 69.927208 74.4) (width 0.5) (layer "F.Cu") (net 2))
+  (segment (start 85.65 67.3) (end 86.852081 67.3) (width 0.5) (layer "F.Cu") (net 2))
   (segment (start 70.941168 63.95) (end 81.03604 63.95) (width 0.5) (layer "F.Cu") (net 2))
-  (segment (start 70.027208 58.55) (end 82.5 58.55) (width 0.5) (layer "F.Cu") (net 2))
+  (segment (start 86.852081 67.3) (end 87.15 67.002081) (width 0.5) (layer "F.Cu") (net 2))
   (segment (start 67.35 70.1) (end 69.85 72.6) (width 0.5) (layer "F.Cu") (net 2))
   (segment (start 67.35 65.2) (end 67.35 64.995584) (width 0.5) (layer "F.Cu") (net 2))
@@
   (segment (start 82.527208 60.35) (end 84.288604 62.111396) (width 0.5) (layer "F.Cu") (net 2))
   (segment (start 80.78604 66.245584) (end 80.290456 65.75) (width 0.5) (layer "F.Cu") (net 2))
+  (segment (start 87.15 62.427208) (end 83.272792 58.55) (width 0.5) (layer "F.Cu") (net 2))
   (segment (start 67.35 67.6) (end 68.638604 68.888604) (width 0.5) (layer "F.Cu") (net 2))
   (segment (start 67.35 67.6) (end 67.35 66.65) (width 0.5) (layer "F.Cu") (net 2))
@@
   (segment (start 67.35 70.1) (end 67.35 67.6) (width 0.5) (layer "F.Cu") (net 2))
   (segment (start 71.341168 69) (end 80.577208 69) (width 0.5) (layer "F.Cu") (net 2))
+  (segment (start 83.272792 58.55) (end 70.027208 58.55) (width 0.5) (layer "F.Cu") (net 2))
   (segment (start 69.420584 67.079416) (end 71.341168 69) (width 0.5) (layer "F.Cu") (net 2))
   (segment (start 69.420584 67.079416) (end 69.83198 66.66802) (width 0.5) (layer "F.Cu") (net 2))
   (segment (start 67.35 71.822792) (end 67.35 70.1) (width 0.5) (layer "F.Cu") (net 2))
+  (segment (start 70.027208 58.55) (end 67.35 61.227208) (width 0.5) (layer "F.Cu") (net 2))
   (segment (start 72.95 67.2) (end 79.831624 67.2) (width 0.5) (layer "F.Cu") (net 2))
   (segment (start 81.454416 70.8) (end 82.202208 70.052208) (width 0.5) (layer "F.Cu") (net 2))
@@
   (segment (start 85.65 71.772792) (end 83.022792 74.4) (width 0.5) (layer "F.Cu") (net 2))
   (segment (start 67.35 66.65) (end 67.35 65.2) (width 0.5) (layer "F.Cu") (net 2))
+  (segment (start 87.15 67.002081) (end 87.15 62.427208) (width 0.5) (layer "F.Cu") (net 2))
   (segment (start 68.684188 68.888604) (end 70.595584 70.8) (width 0.5) (layer "F.Cu") (net 2))
   (segment (start 70.595584 70.8) (end 81.454416 70.8) (width 0.5) (layer "F.Cu") (net 2))
   (segment (start 67.35 65.2) (end 67.35 62.45) (width 0.5) (layer "F.Cu") (net 2))
-  (segment (start 67.35 61.227208) (end 70.027208 58.55) (width 0.5) (layer "F.Cu") (net 2))
   (segment (start 67.35 64.995584) (end 70.195584 62.15) (width 0.5) (layer "F.Cu") (net 2))
   (segment (start 81.781624 62.15) (end 83.690812 64.059188) (width 0.5) (layer "F.Cu") (net 2))

Commit message: ERC DRC
Connections:
- J2 pad 1: Net-(J1-Pin_1) -> unconnected-(J2-Pin_1-Pad1)
- J2 pad 2: Net-(J1-Pin_2) -> unconnected-(J2-Pin_2-Pad2)
Routing:
- net unconnected-(J2-Pin_2-Pad2): track 0.00 -> 185.9 mm
- net Net-(J1-Pin_2): track 185.9 -> 0.00 mm
- net unconnected-(J2-Pin_1-Pad1): track 0.00 -> 137.6 mm
- net Net-(J1-Pin_1): track 137.6 -> 0.00 mm
Changed lines of the file:
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@@
   )
   (net 0 "")
-  (net 1 "Net-(J1-Pin_1)")
-  (net 2 "Net-(J1-Pin_2)")
+  (net 1 "unconnected-(J2-Pin_1-Pad1)")
+  (net 2 "unconnected-(J2-Pin_2-Pad2)")
   (footprint "MountingHole:MountingHole_2.2mm_M2" (layer "F.Cu")
     (at 67.6 74.95)
@@
       (stroke (width 0.1) (type solid)) (layer "F.Fab"))
     (pad "1" thru_hole rect (at 0 0) (size 1.7 1.7) (drill 1) (layers "*.Cu" "*.Mask")
-      (net 1 "Net-(J1-Pin_1)") (pinfunction "Pin_1") (pintype "passive"))
+      (net 1 "unconnected-(J2-Pin_1-Pad1)") (pinfunction "Pin_1") (pintype "passive+no_connect"))
     (pad "2" thru_hole oval (at 0 2.54) (size 1.7 1.7) (drill 1) (layers "*.Cu" "*.Mask")
-      (net 2 "Net-(J1-Pin_2)") (pinfunction "Pin_2") (pintype "passive"))
+      (net 2 "unconnected-(J2-Pin_2-Pad2)") (pinfunction "Pin_2") (pintype "passive+no_connect"))
     (model "${KICAD6_3DMODEL_DIR}/Connector_PinHeader_2.54mm.3dshapes/PinHeader_1x02_P2.54mm_Vertical.wrl" hide
       (offset (xyz 0 0 0))

Commit message: pads
Parts:
- added J1: Conn_01x02, libs:capacitive pads, F.Cu at (74.7, 65.8)
Connections:
- J2 pad 1: unconnected-(J2-Pin_1-Pad1) -> Net-(J1-Pin_1)
- J2 pad 2: unconnected-(J2-Pin_2-Pad2) -> Net-(J1-Pin_2)
Routing:
- net unconnected-(J2-Pin_2-Pad2): track 185.9 -> 0.00 mm
- net unconnected-(J2-Pin_1-Pad1): track 137.6 -> 0.00 mm
- net Net-(J1-Pin_2): track 0.00 -> 116.0 mm, vias 0 -> 2
- net Net-(J1-Pin_1): track 0.00 -> 92.4 mm
Other:
- board text added: "REV1.0"

Commit message: 45mm pad
Parts:
- removed H1, H2, H3, H4: MountingHole, MountingHole:MountingHole_2.2mm_M2
- J1: footprint libs:capacitive pads -> libs:capacitive pads_45x45
- moved J2 72.1 mm to (157.7, 62.0)
- moved J1 59.4 mm to (131.3, 47.6)
Routing:
- net Net-(J1-Pin_1): track 92.4 -> 703.0 mm
- net Net-(J1-Pin_2): track 116.0 -> 595.1 mm, vias 2 -> 0
Other:
- board size 25 x 25 mm -> 52.8 x 46.1 mm
- board text removed: "REV1.0"
