File: lemmy/lemmy.kicad_sch (KiCad schematic)
At the start: 6 parts, among them J1 Conn_01x02, J2 Conn_01x02

Commit message: ERC DRC
Parts:
- removed J1: Conn_01x02, symbol Connector_Generic:Conn_01x02
Connections:
- no-connect marks 0 -> 2
Changed lines of the file:
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@@
 (kicad_sch (version 20230121) (generator eeschema)
   (paper "A4")
-  (wire (pts (xy 58.42 30.48) (xy 53.34 30.48))
-    (stroke (width 0) (type default))
-  )
-  (wire (pts (xy 53.34 30.48) (xy 53.34 38.1))
-    (stroke (width 0) (type default))
-  )
-  (wire (pts (xy 58.42 33.02) (xy 54.61 33.02))
-    (stroke (width 0) (type default))
-  )
-  (wire (pts (xy 53.34 38.1) (xy 58.42 38.1))
-    (stroke (width 0) (type default))
-  )
-  (wire (pts (xy 54.61 40.64) (xy 58.42 40.64))
-    (stroke (width 0) (type default))
-  )
-  (wire (pts (xy 54.61 33.02) (xy 54.61 40.64))
-    (stroke (width 0) (type default))
-  )
-  (symbol (lib_id "Connector_Generic:Conn_01x02") (at 63.5 30.48 0) (unit 1)
-    (in_bom yes) (on_board yes) (dnp no) (fields_autoplaced)
-    (property "Reference" "J1" (at 66.04 31.115 0)
-      (effects (font (size 1.27 1.27)) (justify left))
-    )
-    (property "Value" "Conn_01x02" (at 66.04 33.655 0)
-      (effects (font (size 1.27 1.27)) (justify left))
-    )
-    (property "Footprint" "" (at 63.5 30.48 0)
-      (effects (font (size 1.27 1.27)) hide)
-    )
-    (property "Datasheet" "~" (at 63.5 30.48 0)
-      (effects (font (size 1.27 1.27)) hide)
-    )
-    (pin "1")
-    (pin "2")
-    (instances
-      (project "lemmy"
-        (path "/675439b2-a86f-45f3-a389-b5122f62382e"
-          (reference "J1") (unit 1)
-        )
-      )
-    )
-  )
+  (no_connect (at 58.42 38.1))
+  (no_connect (at 58.42 40.64))
   (symbol (lib_id "Mechanical:MountingHole") (at 92.71 29.21 0) (unit 1)
     (in_bom yes) (on_board yes) (dnp no) (fields_autoplaced)

Commit message: pads
Parts:
- added J1: Conn_01x02, libs:capacitive pads, symbol Connector_Generic:Conn_01x02
Connections:
- net at J2.1 (Pin_1): now also J1.1 (Pin_1)
- net at J2.2 (Pin_2): now also J1.2 (Pin_2)
- no-connect marks 2 -> 0
Changed lines of the file:
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@@
 (kicad_sch (version 20230121) (generator eeschema)
   (paper "A4")
-  (no_connect (at 58.42 38.1))
-  (no_connect (at 58.42 40.64))
+  (wire (pts (xy 58.42 30.48) (xy 53.34 30.48))
+    (stroke (width 0) (type default))
+  )
+  (wire (pts (xy 53.34 30.48) (xy 53.34 38.1))
+    (stroke (width 0) (type default))
+  )
+  (wire (pts (xy 58.42 33.02) (xy 54.61 33.02))
+    (stroke (width 0) (type default))
+  )
+  (wire (pts (xy 53.34 38.1) (xy 58.42 38.1))
+    (stroke (width 0) (type default))
+  )
+  (wire (pts (xy 54.61 40.64) (xy 58.42 40.64))
+    (stroke (width 0) (type default))
+  )
+  (wire (pts (xy 54.61 33.02) (xy 54.61 40.64))
+    (stroke (width 0) (type default))
+  )
+  (symbol (lib_id "Connector_Generic:Conn_01x02") (at 63.5 30.48 0) (unit 1)
+    (in_bom yes) (on_board yes) (dnp no) (fields_autoplaced)
+    (property "Reference" "J1" (at 66.04 31.115 0)
+      (effects (font (size 1.27 1.27)) (justify left))
+    )
+    (property "Value" "Conn_01x02" (at 66.04 33.655 0)
+      (effects (font (size 1.27 1.27)) (justify left))
+    )
+    (property "Footprint" "libs:capacitive pads" (at 63.5 30.48 0)
+      (effects (font (size 1.27 1.27)) hide)
+    )
+    (property "Datasheet" "~" (at 63.5 30.48 0)
+      (effects (font (size 1.27 1.27)) hide)
+    )
+    (pin "1")
+    (pin "2")
+    (instances
+      (project "lemmy"
+        (path "/675439b2-a86f-45f3-a389-b5122f62382e"
+          (reference "J1") (unit 1)
+        )
+      )
+    )
+  )
   (symbol (lib_id "Mechanical:MountingHole") (at 92.71 29.21 0) (unit 1)
     (in_bom yes) (on_board yes) (dnp no) (fields_autoplaced)

Commit message: 45mm pad
Parts:
- J1: footprint libs:capacitive pads -> libs:capacitive pads_45x45
Changed lines of the file:
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@@
       (effects (font (size 1.27 1.27)) (justify left))
     )
-    (property "Footprint" "libs:capacitive pads" (at 63.5 30.48 0)
+    (property "Footprint" "libs:capacitive pads_45x45" (at 63.5 30.48 0)
       (effects (font (size 1.27 1.27)) hide)
     )
